File: il300 LM358 VM daughter board.kicad_sch (KiCad schematic)
At the start: 13 parts, among them J1 Screw_Terminal_01x08, U1 LM358, U2 IL300, U3 IL300, U4 LM358

Commit message: Update schematics
Parts:
- removed J1: Screw_Terminal_01x08, TerminalBlock_Phoenix:TerminalBlock_Phoenix_PT-1,5-8-3.5-H_1x08_P3.50mm_Horizontal, symbol Connector:Screw_Terminal_01x08
- added J1, J2: Screw_Terminal_01x04, symbol Connector:Screw_Terminal_01x04
- added R6, R7: 100R, symbol Device:R
Connections:
- net 12V_IN: now also J1.1 (Pin_1)
- net 5V(MCU): now also J2.1 (Pin_1)
- net GND: now also J1.2 (Pin_2)
- net GNDREF: now also J2.2 (Pin_2)
- net SIG_IN_1: now also J1.3 (Pin_3)
- net SIG_IN_2: now also J1.4 (Pin_4)
- net SIG_OUT_1: now also J2.3 (Pin_3)
- net SIG_OUT_2: now also J2.4 (Pin_4)
- net at U3.2: now also R7.1; no longer U1.7
- net at U2.2: now also R6.1; no longer U1.1
- new net: R7.2, U1.7
- new net: R6.2, U1.1
Other:
- moved on the sheet: C1, C2, C3, C4, R2, R3, R4, R5, U1A, U1B, U1C, U2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

Commit message: Update schematics
Parts:
- removed J1, J2: Screw_Terminal_01x04, symbol Connector:Screw_Terminal_01x04
- added J1: Screw_Terminal_01x08, symbol Connector:Screw_Terminal_01x08
Connections:
- net 12V_IN: now also J1.1 (Pin_1)
- net 5V(MCU): now also J1.5 (Pin_5)
- net GND: now also J1.2 (Pin_2)
- net GNDREF: now also J1.6 (Pin_6)
- net SIG_IN_1: now also J1.3 (Pin_3)
- net SIG_IN_2: now also J1.4 (Pin_4)
- net SIG_OUT_1: now also J1.7 (Pin_7)
- net SIG_OUT_2: now also J1.8 (Pin_8)
Changed lines of the file:
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@@
     (stroke (width 0) (type default))
   )
-  (wire (pts (xy 58.42 128.27) (xy 69.85 128.27))
+  (wire (pts (xy 59.69 115.57) (xy 71.12 115.57))
     (stroke (width 0) (type default))
   )
@@
     (stroke (width 0) (type default))
   )
-  (wire (pts (xy 58.42 123.19) (xy 69.85 123.19))
+  (wire (pts (xy 59.69 110.49) (xy 71.12 110.49))
     (stroke (width 0) (type default))
   )
@@
     (stroke (width 0) (type default))
   )
-  (wire (pts (xy 58.42 130.81) (xy 69.85 130.81))
+  (wire (pts (xy 59.69 118.11) (xy 71.12 118.11))
     (stroke (width 0) (type default))
   )
@@
     (effects (font (size 1.27 1.27)) (justify right bottom))
   )
-  (label "5V(MCU)" (at 69.85 123.19 0) (fields_autoplaced)
+  (label "5V(MCU)" (at 71.12 110.49 0) (fields_autoplaced)
     (effects (font (size 1.27 1.27)) (justify left bottom))
   )
@@
     (effects (font (size 1.27 1.27)) (justify left bottom))
   )
-  (label "SIG_OUT_1" (at 69.85 128.27 0) (fields_autoplaced)
+  (label "SIG_OUT_1" (at 71.12 115.57 0) (fields_autoplaced)
     (effects (font (size 1.27 1.27)) (justify left bottom))
   )
@@
     (effects (font (size 1.27 1.27)) (justify left bottom))
   )
-  (label "SIG_OUT_2" (at 69.85 130.81 0) (fields_autoplaced)
+  (label "SIG_OUT_2" (at 71.12 118.11 0) (fields_autoplaced)
     (effects (font (size 1.27 1.27)) (justify left bottom))
   )
@@
         (path "/8691f7a3-8fa1-49ca-9374-de1c4f2f2cbe"
           (reference "R7") (unit 1)
+        )
+      )
+    )
+  )
+  (symbol (lib_id "Connector:Screw_Terminal_01x08") (at 54.61 107.95 0) (mirror y) (unit 1)
+    (in_bom yes) (on_board yes) (dnp no) (fields_autoplaced)
+    (property "Reference" "J1" (at 54.61 93.98 0)
+      (effects (font (size 1.27 1.27)))
+    )
+    (property "Value" "Screw_Terminal_01x08" (at 54.61 96.52 0)
+      (effects (font (size 1.27 1.27)))
+    )
+    (property "Footprint" "" (at 54.61 107.95 0)
+      (effects (font (size 1.27 1.27)) hide)
+    )
+    (property "Datasheet" "~" (at 54.61 107.95 0)
+      (effects (font (size 1.27 1.27)) hide)
+    )
+    (pin "1")
+    (pin "7")
+    (pin "4")
+    (pin "8")
+    (pin "3")
+    (pin "5")
+    (pin "6")
+    (pin "2")
+    (instances
+      (project "il300 LM358 VM daughter board"
+        (path "/8691f7a3-8fa1-49ca-9374-de1c4f2f2cbe"
+          (reference "J1") (unit 1)
         )
       )
@@
     )
   )
-  (symbol (lib_id "power:GNDREF") (at 58.42 125.73 90) (unit 1)
-    (in_bom yes) (on_board yes) (dnp no) (fields_autoplaced)
-    (property "Reference" "#PWR010" (at 64.77 125.73 0)
-      (effects (font (size 1.27 1.27)) hide)
-    )
-    (property "Value" "GNDREF" (at 62.23 125.73 90)
-      (effects (font (size 1.27 1.27)) (justify right))
-    )
-    (property "Footprint" "" (at 58.42 125.73 0)
-      (effects (font (size 1.27 1.27)) hide)
-    )
-    (property "Datasheet" "" (at 58.42 125.73 0)
+  (symbol (lib_id "power:GNDREF") (at 59.69 113.03 90) (unit 1)
+    (in_bom yes) (on_board yes) (dnp no) (fields_autoplaced)
+    (property "Reference" "#PWR010" (at 66.04 113.03 0)
+      (effects (font (size 1.27 1.27)) hide)
+    )
+    (property "Value" "GNDREF" (at 63.5 113.03 90)
+      (effects (font (size 1.27 1.27)) (justify right))
+    )
+    (property "Footprint" "" (at 59.69 113.03 0)
+      (effects (font (size 1.27 1.27)) hide)
+    )
+    (property "Datasheet" "" (at 59.69 113.03 0)
       (effects (font (size 1.27 1.27)) hide)
     )
@@
         (path "/8691f7a3-8fa1-49ca-9374-de1c4f2f2cbe"
           (reference "R4") (unit 1)
-        )
-      )
-    )
-  )
-  (symbol (lib_id "Connector:Screw_Terminal_01x04") (at 53.34 125.73 0) (mirror y) (unit 1)
-    (in_bom yes) (on_board yes) (dnp no) (fields_autoplaced)
-    (property "Reference" "J2" (at 53.34 116.84 0)
-      (effects (font (size 1.27 1.27)))
-    )
-    (property "Value" "Screw_Terminal_01x04" (at 53.34 119.38 0)
-      (effects (font (size 1.27 1.27)))
-    )
-    (property "Footprint" "" (at 53.34 125.73 0)
-      (effects (font (size 1.27 1.27)) hide)
-    )
-    (property "Datasheet" "~" (at 53.34 125.73 0)
-      (effects (font (size 1.27 1.27)) hide)
-    )
-    (pin "3")
-    (pin "1")
-    (pin "2")
-    (pin "4")
-    (instances
-      (project "il300 LM358 VM daughter board"
-        (path "/8691f7a3-8fa1-49ca-9374-de1c4f2f2cbe"
-          (reference "J2") (unit 1)
         )
       )
@@
         )
       )
-    )
-  )
-  (symbol (lib_id "Connector:Screw_Terminal_01x04") (at 54.61 102.87 0) (mirror y) (unit 1)
-    (in_bom yes) (on_board yes) (dnp no) (fields_autoplaced)
-    (property "Reference" "J1" (at 54.61 93.98 0)
-      (effects (font (size 1.27 1.27)))
-    )
-    (property "Value" "Screw_Terminal_01x04" (at 54.61 96.52 0)
-      (effects (font (size 1.27 1.27)))
-    )
-    (property "Footprint" "" (at 54.61 102.87 0)
-      (effects (font (size 1.27 1.27)) hide)
-    )
-    (property "Datasheet" "~" (at 54.61 102.87 0)
-      (effects (font (size 1.27 1.27)) hide)
-    )
-    (pin "3")
-    (pin "1")
-    (pin "2")
-    (pin "4")
-    (instances
-      (project "il300 LM358 VM daughter board"
-        (path "/8691f7a3-8fa1-49ca-9374-de1c4f2f2cbe"
-          (reference "J1") (unit 1)
-        )
-      )

Commit message: Update schematics
Connections:
- net 12V_IN: now also J1.5 (Pin_5); no longer J1.1 (Pin_1)
- net 5V(MCU): now also J1.1 (Pin_1); no longer J1.5 (Pin_5)
- net GND: now also J1.6 (Pin_6); no longer J1.2 (Pin_2)
- net GNDREF: now also J1.2 (Pin_2); no longer J1.6 (Pin_6)
- net SIG_IN_1: now also J1.7 (Pin_7); no longer J1.3 (Pin_3)
- net SIG_IN_2: now also J1.8 (Pin_8); no longer J1.4 (Pin_4)
- net SIG_OUT_1: now also J1.3 (Pin_3); no longer J1.7 (Pin_7)
- net SIG_OUT_2: now also J1.4 (Pin_4); no longer J1.8 (Pin_8)

Commit message: Added schematics
Parts:
- C1, C2, C3, C4: footprint (none) -> Capacitor_SMD:C_1206_3216Metric
- J1: footprint (none) -> TerminalBlock_Phoenix:TerminalBlock_Phoenix_MPT-0,5-8-2.54_1x08_P2.54mm_Horizontal
- R2, R3, R4, R5, R6, R7: footprint (none) -> Resistor_SMD:R_1206_3216Metric
- U1, U2, U3, U4: footprint (none) -> Package_SO:SOIC-8_3.9x4.9mm_P1.27mm
Connections:
- net 5V(MCU): now also J1.3 (Pin_3); no longer J1.1 (Pin_1)
- net GNDREF: now also J1.4 (Pin_4); no longer J1.2 (Pin_2)
- net SIG_OUT_1: now also J1.1 (Pin_1); no longer J1.3 (Pin_3)
- net SIG_OUT_2: now also J1.2 (Pin_2); no longer J1.4 (Pin_4)
Changed lines of the file:
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@@
+    (stroke (width 0) (type default))
+  )
+  (wire (pts (xy 59.69 102.87) (xy 62.23 102.87))
     (stroke (width 0) (type default))
   )
@@
     (stroke (width 0) (type default))
   )
-  (wire (pts (xy 59.69 100.33) (xy 71.12 100.33))
+  (wire (pts (xy 76.2 106.68) (xy 71.12 106.68))
+    (stroke (width 0) (type default))
+  )
+  (wire (pts (xy 59.69 100.33) (xy 73.66 100.33))
     (stroke (width 0) (type default))
   )
@@
   )
   (wire (pts (xy 137.16 120.65) (xy 137.16 124.46))
+    (stroke (width 0) (type default))
+  )
+  (wire (pts (xy 71.12 106.68) (xy 71.12 107.95))
     (stroke (width 0) (type default))
   )
@@
     (effects (font (size 1.27 1.27)) (justify right bottom))
   )
-  (label "5V(MCU)" (at 71.12 100.33 0) (fields_autoplaced)
+  (label "5V(MCU)" (at 71.12 105.41 0) (fields_autoplaced)
     (effects (font (size 1.27 1.27)) (justify left bottom))
   )
@@
     (effects (font (size 1.27 1.27)) (justify left bottom))
   )
-  (label "SIG_OUT_1" (at 71.12 105.41 0) (fields_autoplaced)
+  (label "SIG_OUT_1" (at 73.66 100.33 0) (fields_autoplaced)
     (effects (font (size 1.27 1.27)) (justify left bottom))
   )
@@
     (effects (font (size 1.27 1.27)) (justify left bottom))
   )
-  (label "SIG_OUT_2" (at 71.12 107.95 0) (fields_autoplaced)
+  (label "SIG_OUT_2" (at 62.23 102.87 0) (fields_autoplaced)
     (effects (font (size 1.27 1.27)) (justify left bottom))
   )
@@
       (effects (font (size 1.27 1.27)))
     )
-    (property "Footprint" "" (at 160.02 109.982 90)
+    (property "Footprint" "Resistor_SMD:R_1206_3216Metric" (at 160.02 109.982 90)
       (effects (font (size 1.27 1.27)) hide)
     )
@@
       (effects (font (size 1.27 1.27)))
     )
-    (property "Footprint" "" (at 54.61 107.95 0)
+    (property "Footprint" "TerminalBlock_Phoenix:TerminalBlock_Phoenix_MPT-0,5-8-2.54_1x08_P2.54mm_Horizontal" (at 54.61 107.95 0)
       (effects (font (size 1.27 1.27)) hide)
     )
@@
       (effects (font (size 1.27 1.27)))
     )
-    (property "Footprint" "" (at 156.21 57.912 90)
+    (property "Footprint" "Resistor_SMD:R_1206_3216Metric" (at 156.21 57.912 90)
       (effects (font (size 1.27 1.27)) hide)
     )
@@
       (effects (font (size 1.27 1.27)))
     )
-    (property "Footprint" "" (at 144.78 118.11 0)
+    (property "Footprint" "Package_SO:SOIC-8_3.9x4.9mm_P1.27mm" (at 144.78 118.11 0)
       (effects (font (size 1.27 1.27)) hide)
     )
@@
       (effects (font (size 1.27 1.27)))
     )
-    (property "Footprint" "" (at 165.1 59.69 0)
+    (property "Footprint" "Package_SO:SOIC-8_3.9x4.9mm_P1.27mm" (at 165.1 59.69 0)
       (effects (font (size 1.27 1.27)) (justify left) hide)
     )
@@
       (effects (font (size 1.27 1.27)) (justify right))
     )
-    (property "Footprint" "" (at 185.928 130.81 90)
+    (property "Footprint" "Resistor_SMD:R_1206_3216Metric" (at 185.928 130.81 90)
       (effects (font (size 1.27 1.27)) hide)
     )
@@
       (effects (font (size 1.27 1.27)))
     )
-    (property "Footprint" "" (at 138.43 59.69 0)
+    (property "Footprint" "Package_SO:SOIC-8_3.9x4.9mm_P1.27mm" (at 138.43 59.69 0)
       (effects (font (size 1.27 1.27)) hide)
     )
@@
     )
   )
-  (symbol (lib_id "power:GNDREF") (at 59.69 102.87 90) (unit 1)
-    (in_bom yes) (on_board yes) (dnp no) (fields_autoplaced)
-    (property "Reference" "#PWR010" (at 66.04 102.87 0)
-      (effects (font (size 1.27 1.27)) hide)
-    )
-    (property "Value" "GNDREF" (at 63.5 102.87 90)
-      (effects (font (size 1.27 1.27)) (justify right))
-    )
-    (property "Footprint" "" (at 59.69 102.87 0)
-      (effects (font (size 1.27 1.27)) hide)
-    )
-    (property "Datasheet" "" (at 59.69 102.87 0)
+  (symbol (lib_id "power:GNDREF") (at 76.2 106.68 90) (unit 1)
+    (in_bom yes) (on_board yes) (dnp no)
+    (property "Reference" "#PWR010" (at 82.55 106.68 0)
+      (effects (font (size 1.27 1.27)) hide)
+    )
+    (property "Value" "GNDREF" (at 80.01 106.68 90)
+      (effects (font (size 1.27 1.27)) (justify right))
+    )
+    (property "Footprint" "" (at 76.2 106.68 0)
+      (effects (font (size 1.27 1.27)) hide)
+    )
+    (property "Datasheet" "" (at 76.2 106.68 0)
       (effects (font (size 1.27 1.27)) hide)
     )
@@
       (effects (font (size 1.27 1.27)) (justify left))
     )
-    (property "Footprint" "" (at 161.5948 129.54 0)
+    (property "Footprint" "Capacitor_SMD:C_1206_3216Metric" (at 161.5948 129.54 0)
       (effects (font (size 1.27 1.27)) hide)
     )
@@
       (effects (font (size 1.27 1.27)) (justify left))
     )
-    (property "Footprint" "" (at 161.5948 77.47 0)
+    (property "Footprint" "Capacitor_SMD:C_1206_3216Metric" (at 161.5948 77.47 0)
       (effects (font (size 1.27 1.27)) hide)
     )
@@
       (effects (font (size 1.27 1.27)) (justify left))
     )
-    (property "Footprint" "" (at 185.7248 121.92 0)
+    (property "Footprint" "Capacitor_SMD:C_1206_3216Metric" (at 185.7248 121.92 0)
       (effects (font (size 1.27 1.27)) hide)
     )
@@
       (effects (font (size 1.27 1.27)) (justify right))
     )
-    (property "Footprint" "" (at 187.198 76.2 90)
+    (property "Footprint" "Resistor_SMD:R_1206_3216Metric" (at 187.198 76.2 90)
       (effects (font (size 1.27 1.27)) hide)
     )
@@
       (effects (font (size 1.27 1.27)) (justify right))
     )
-    (property "Footprint" "" (at 138.938 129.54 90)
+    (property "Footprint" "Resistor_SMD:R_1206_3216Metric" (at 138.938 129.54 90)
       (effects (font (size 1.27 1.27)) hide)
     )
@@
       (effects (font (size 1.27 1.27)) (justify right))
     )
-    (property "Footprint" "" (at 242.57 100.33 0)
+    (property "Footprint" "Package_SO:SOIC-8_3.9x4.9mm_P1.27mm" (at 242.57 100.33 0)
       (effects (font (size 1.27 1.27)) hide)
     )
@@
       (effects (font (size 1.27 1.27)))
     )
-    (property "Footprint" "" (at 166.37 111.76 0)
+    (property "Footprint" "Package_SO:SOIC-8_3.9x4.9mm_P1.27mm" (at 166.37 111.76 0)
       (effects (font (size 1.27 1.27)) (justify left) hide)
     )
@@
       (effects (font (size 1.27 1.27)))
     )
-    (property "Footprint" "" (at 204.47 120.65 0)
+    (property "Footprint" "Package_SO:SOIC-8_3.9x4.9mm_P1.27mm" (at 204.47 120.65 0)
       (effects (font (size 1.27 1.27)) hide)
     )
@@
       (effects (font (size 1.27 1.27)) (justify left))
     )
-    (property "Footprint" "" (at 185.7248 57.15 0)
+    (property "Footprint" "Capacitor_SMD:C_1206_3216Metric" (at 185.7248 57.15 0)
       (effects (font (size 1.27 1.27)) hide)
     )
@@
       (effects (font (size 1.27 1.27)) (justify right))
     )
-    (property "Footprint" "" (at 132.588 69.85 90)
+    (property "Footprint" "Resistor_SMD:R_1206_3216Metric" (at 132.588 69.85 90)
       (effects (font (size 1.27 1.27)) hide)
     )
@@
       (effects (font (size 1.27 1.27)))
     )
-    (property "Footprint" "" (at 200.66 67.31 0)
+    (property "Footprint" "Package_SO:SOIC-8_3.9x4.9mm_P1.27mm" (at 200.66 67.31 0)
       (effects (font (size 1.27 1.27)) hide)
     )
@@
       (effects (font (size 1.27 1.27)) (justify left))
     )
-    (property "Footprint" "" (at 101.6 102.87 0)
-      (effects (font (size 1.27 1.27)) hide)
-    )
+    (property "Footprint" "Package_SO:SOIC-8_3.9x4.9mm_P1.27mm" (at 101.6 102.87 0)
+      (effects (font (size 1.27 1.27)) hide)
+    )
